File: électronique/KiCad/bigmax_hat/bigmax_hat.kicad_pcb (KiCad board)
At the start: 2 copper layers, 94 x 76.8 mm, 6 parts, among them J1 Conn_01x02, J2 Conn_01x03, U1 jsumo_micro_start, U2 generic_18650_3s_case, U3 generic_bms_3s_10A, U4 generic_vertical_slide_switch

Commit message: first 22 push
Other:
- net class Default removed
